File: PCB/sub_module/sub_module.sch (EAGLE design)
At the start: 11 parts, among them J1 J7MM, J2 J7MM, X1 DCJACK-MJ179P-R

Commit message: sub_moduleを改良
Parts:
- removed D1: BAT49, diode:BAT49
- added J3: J15MM, jumper:J15MM
- added JP3, JP4: (no value), jumper:JP2E
- added R1: 4.7k, rcl:R-US_0207/2V
- U$1: value CR2032-HOLDER -> CR2032-HOLDER2; device CR2032-holder:CR2032-HOLDER -> CR2032-holder:CR2032-HOLDER2
- X1: value DCJACK-MJ179P-R -> DCJACK-PJ102-R; device dcjack:DCJACK-MJ179P-R -> dcjack:DCJACK-PJ102-R
Connections:
- new net N$10: JP3.1, U$2.PWM/DP24
- new net N$4: JP4.3, U$2.SERAL_RX/DP15
- new net N$7: JP4.2, U$2.SERIAL_TX/DP16
- new net N$8: J3.1, JP1.4
- new net N$9: JP3.2, R1.1, U$2.NR/DP23
- net GND: now also JP3.3, R1.2
- net N$2: now also J3.2; no longer JP1.4
- net VCC: now also U$1.+3V; no longer D1.C, U$1.3VR
- net VDD: now also JP4.1; no longer D1.A
Other:
- moved on the sheet: J2, JP2
Changed lines of the file:
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@@
 <?xml version="1.0" encoding="utf-8"?>
 <!DOCTYPE eagle SYSTEM "eagle.dtd">
-<eagle version="7.6.0">
+<eagle version="7.5.0">
 <drawing>
 <settings>
@@
 </classes>
 <parts>
-<part name="U$1" library="CR2032-holder" deviceset="CR2032-HOLDER" device=""/>
 <part name="SUPPLY1" library="supply2" deviceset="GND" device=""/>
 <part name="SUPPLY2" library="supply2" deviceset="VCC" device=""/>
 <part name="SUPPLY3" library="supply2" deviceset="VCC" device=""/>
 <part name="SUPPLY4" library="supply2" deviceset="VDD" device=""/>
-<part name="X1" library="dcjack" deviceset="DCJACK" device="-MJ179P-R"/>
+<part name="X1" library="dcjack" deviceset="DCJACK" device="-PJ102-R" value="DCJACK-PJ102-R"/>
 <part name="SUPPLY5" library="supply2" deviceset="GND" device=""/>
 <part name="SUPPLY6" library="supply2" deviceset="VDD" device=""/>
-<part name="D1" library="diode" deviceset="BAT49" device=""/>
 <part name="JP1" library="jumper" deviceset="JP4E" device=""/>
 <part name="SUPPLY8" library="supply2" deviceset="GND" device=""/>
@@
 <part name="SUPPLY15" library="supply2" deviceset="GND" device=""/>
 <part name="J2" library="jumper" deviceset="J" device="7MM" value="J7MM"/>
+<part name="U$1" library="CR2032-holder" deviceset="CR2032-HOLDER2" device=""/>
+<part name="JP3" library="jumper" deviceset="JP2E" device=""/>
+<part name="JP4" library="jumper" deviceset="JP2E" device=""/>
+<part name="SUPPLY16" library="supply2" deviceset="VDD" device=""/>
+<part name="SUPPLY17" library="supply2" deviceset="GND" device=""/>
+<part name="R1" library="rcl" deviceset="R-US_" device="0207/2V" value="4.7k"/>
+<part name="J3" library="jumper" deviceset="J" device="15MM" value="J15MM"/>
 </parts>
 <sheets>
@@
 </plain>
 <instances>
-<instance part="U$1" gate="G$1" x="2.54" y="58.42" rot="R270"/>
 <instance part="SUPPLY1" gate="GND" x="2.54" y="50.8"/>
 <instance part="SUPPLY2" gate="G$1" x="0" y="78.74"/>
@@
 <instance part="SUPPLY5" gate="GND" x="-17.78" y="50.8"/>
 <instance part="SUPPLY6" gate="G$1" x="-17.78" y="78.74"/>
-<instance part="D1" gate="A" x="22.86" y="73.66" rot="R180"/>
 <instance part="JP1" gate="G$1" x="45.72" y="71.12"/>
 <instance part="SUPPLY8" gate="GND" x="48.26" y="50.8"/>
@@
 <instance part="SUPPLY14" gate="G$1" x="20.32" y="58.42"/>
 <instance part="J1" gate="1" x="104.14" y="101.6" rot="R90"/>
-<instance part="JP2" gate="1" x="152.4" y="99.06"/>
-<instance part="SUPPLY11" gate="G$1" x="142.24" y="109.22"/>
-<instance part="SUPPLY15" gate="GND" x="152.4" y="88.9"/>
-<instance part="J2" gate="1" x="142.24" y="101.6" rot="R90"/>
+<instance part="JP2" gate="1" x="175.26" y="45.72"/>
+<instance part="SUPPLY11" gate="G$1" x="162.56" y="58.42"/>
+<instance part="SUPPLY15" gate="GND" x="175.26" y="25.4"/>
+<instance part="J2" gate="1" x="162.56" y="48.26" rot="R90"/>
+<instance part="U$1" gate="G$1" x="2.54" y="60.96" rot="R270"/>
+<instance part="JP3" gate="1" x="83.82" y="111.76"/>
+<instance part="JP4" gate="1" x="129.54" y="101.6"/>
+<instance part="SUPPLY16" gate="G$1" x="124.46" y="111.76"/>
+<instance part="SUPPLY17" gate="GND" x="86.36" y="99.06"/>
+<instance part="R1" gate="G$1" x="93.98" y="96.52" rot="R90"/>
+<instance part="J3" gate="1" x="53.34" y="78.74" rot="R90"/>
 </instances>
 <busses>
@@
 <net name="GND" class="0">
 <segment>
-<pinref part="U$1" gate="G$1" pin="GND"/>
-<pinref part="SUPPLY1" gate="GND" pin="GND"/>
-</segment>
-<segment>
 <pinref part="X1" gate="G$1" pin="3"/>
 <pinref part="X1" gate="G$1" pin="2"/>
@@
 <pinref part="SUPPLY9" gate="GND" pin="GND"/>
 <pinref part="C1" gate="G$1" pin="2"/>
-<wire x1="96.52" y1="106.68" x2="96.52" y2="91.44" width="0.1524" layer="91"/>
+<wire x1="96.52" y1="106.68" x2="96.52" y2="101.6" width="0.1524" layer="91"/>
+<wire x1="96.52" y1="101.6" x2="96.52" y2="91.44" width="0.1524" layer="91"/>
 <wire x1="96.52" y1="91.44" x2="96.52" y2="86.36" width="0.1524" layer="91"/>
 <pinref part="U$2" gate="G$1" pin="GND"/>
 <wire x1="96.52" y1="86.36" x2="99.06" y2="86.36" width="0.1524" layer="91"/>
 <wire x1="99.06" y1="86.36" x2="99.06" y2="83.82" width="0.1524" layer="91"/>
+<pinref part="R1" gate="G$1" pin="2"/>
+<wire x1="93.98" y1="101.6" x2="96.52" y2="101.6" width="0.1524" layer="91"/>
 </segment>
 <segment>
@@
 <segment>
 <pinref part="JP2" gate="1" pin="2"/>
-<wire x1="152.4" y1="96.52" x2="152.4" y2="91.44" width="0.1524" layer="91"/>
+<wire x1="175.26" y1="43.18" x2="175.26" y2="27.94" width="0.1524" layer="91"/>
 <pinref part="SUPPLY15" gate="GND" pin="GND"/>
+</segment>
+<segment>
+<pinref part="SUPPLY1" gate="GND" pin="GND"/>
+<pinref part="U$1" gate="G$1" pin="GND"/>
+</segment>
+<segment>
+<pinref part="JP3" gate="1" pin="3"/>
+<pinref part="SUPPLY17" gate="GND" pin="GND"/>
+<wire x1="86.36" y1="109.22" x2="86.36" y2="101.6" width="0.1524" layer="91"/>
 </segment>
 </net>
@@
 <pinref part="SUPPLY3" gate="G$1" pin="VCC"/>
 <wire x1="17.78" y1="76.2" x2="17.78" y2="73.66" width="0.1524" layer="91"/>
-<pinref part="D1" gate="A" pin="C"/>
 <wire x1="17.78" y1="73.66" x2="20.32" y2="73.66" width="0.1524" layer="91"/>
 </segment>
 <segment>
 <pinref part="SUPPLY2" gate="G$1" pin="VCC"/>
-<pinref part="U$1" gate="G$1" pin="3VR"/>
 <wire x1="0" y1="76.2" x2="5.08" y2="76.2" width="0.1524" layer="91"/>
 <wire x1="5.08" y1="76.2" x2="5.08" y2="71.12" width="0.1524" layer="91"/>
+<pinref part="U$1" gate="G$1" pin="+3V"/>
+<wire x1="5.08" y1="71.12" x2="2.54" y2="71.12" width="0.1524" layer="91"/>
+<wire x1="2.54" y1="71.12" x2="2.54" y2="68.58" width="0.1524" layer="91"/>
 </segment>
 <segment>
@@
 <pinref part="SUPPLY4" gate="G$1" pin="VDD"/>
 <wire x1="27.94" y1="76.2" x2="27.94" y2="73.66" width="0.1524" layer="91"/>
-<pinref part="D1" gate="A" pin="A"/>
 <wire x1="27.94" y1="73.66" x2="25.4" y2="73.66" width="0.1524" layer="91"/>
 <wire x1="27.94" y1="73.66" x2="27.94" y2="68.58" width="0.1524" layer="91"/>
@@
 <pinref part="SUPPLY11" gate="G$1" pin="VDD"/>
 <pinref part="J2" gate="1" pin="2"/>
+<wire x1="162.56" y1="53.34" x2="162.56" y2="55.88" width="0.1524" layer="91"/>
+</segment>
+<segment>
+<pinref part="JP4" gate="1" pin="1"/>
+<wire x1="127" y1="99.06" x2="124.46" y2="99.06" width="0.1524" layer="91"/>
+<wire x1="124.46" y1="99.06" x2="124.46" y2="109.22" width="0.1524" layer="91"/>
+<pinref part="SUPPLY16" gate="G$1" pin="VDD"/>
 </segment>
 </net>
@@
 <pinref part="IC1" gate="G$1" pin="SDA"/>
 <wire x1="88.9" y1="27.94" x2="55.88" y2="27.94" width="0.1524" layer="91"/>
-<wire x1="55.88" y1="27.94" x2="55.88" y2="68.58" width="0.1524" layer="91"/>
-<pinref part="JP1" gate="G$1" pin="4"/>
-<wire x1="55.88" y1="68.58" x2="55.88" y2="93.98" width="0.1524" layer="91"/>
-<wire x1="50.8" y1="68.58" x2="55.88" y2="68.58" width="0.1524" layer="91"/>
+<wire x1="55.88" y1="27.94" x2="55.88" y2="83.82" width="0.1524" layer="91"/>
+<pinref part="J3" gate="1" pin="2"/>
+<wire x1="55.88" y1="83.82" x2="55.88" y2="93.98" width="0.1524" layer="91"/>
+<wire x1="53.34" y1="83.82" x2="55.88" y2="83.82" width="0.1524" layer="91"/>
 </segment>
 </net>
@@
 <wire x1="104.14" y1="96.52" x2="104.14" y2="91.44" width="0.1524" layer="91"/>
 <pinref part="C1" gate="G$1" pin="1"/>
+<junction x="104.14" y="91.44"/>
 <wire x1="104.14" y1="91.44" x2="104.14" y2="83.82" width="0.1524" layer="91"/>
-<junction x="104.14" y="91.44"/>
 </segment>
 </net>
@@
 <pinref part="U$2" gate="G$1" pin="DP13/AN"/>
 <wire x1="129.54" y1="33.02" x2="129.54" y2="30.48" width="0.1524" layer="91"/>
-<wire x1="129.54" y1="30.48" x2="154.94" y2="30.48" width="0.1524" layer="91"/>
-<wire x1="154.94" y1="30.48" x2="154.94" y2="96.52" width="0.1524" layer="91"/>
+<wire x1="129.54" y1="30.48" x2="177.8" y2="30.48" width="0.1524" layer="91"/>
+<wire x1="177.8" y1="30.48" x2="177.8" y2="43.18" width="0.1524" layer="91"/>
 </segment>
 </net>
@@
 <segment>
 <pinref part="JP2" gate="1" pin="1"/>
-<wire x1="149.86" y1="96.52" x2="142.24" y2="96.52" width="0.1524" layer="91"/>
+<wire x1="172.72" y1="43.18" x2="162.56" y2="43.18" width="0.1524" layer="91"/>
 <pinref part="J2" gate="1" pin="1"/>
 </segment>
 </net>
+<net name="N$7" class="0">
+<segment>
+<pinref part="JP4" gate="1" pin="2"/>
+<pinref part="U$2" gate="G$1" pin="SERIAL_TX/DP16"/>
+<wire x1="129.54" y1="99.06" x2="129.54" y2="83.82" width="0.1524" layer="91"/>
+</segment>
+</net>
+<net name="N$4" class="0">
+<segment>
+<pinref part="JP4" gate="1" pin="3"/>
+<pinref part="U$2" gate="G$1" pin="SERAL_RX/DP15"/>
+<wire x1="132.08" y1="99.06" x2="134.62" y2="99.06" width="0.1524" layer="91"/>
+<wire x1="134.62" y1="99.06" x2="134.62" y2="83.82" width="0.1524" layer="91"/>
+</segment>
+</net>
+<net name="N$9" class="0">
+<segment>
+<pinref part="JP3" gate="1" pin="2"/>
+<wire x1="83.82" y1="109.22" x2="83.82" y2="91.44" width="0.1524" layer="91"/>
+<pinref part="U$2" gate="G$1" pin="NR/DP23"/>
+<wire x1="83.82" y1="91.44" x2="93.98" y2="91.44" width="0.1524" layer="91"/>
+<wire x1="93.98" y1="91.44" x2="93.98" y2="83.82" width="0.1524" layer="91"/>
+<pinref part="R1" gate="G$1" pin="1"/>
+<junction x="93.98" y="91.44"/>
+</segment>
+</net>
+<net name="N$10" class="0">
+<segment>
+<pinref part="U$2" gate="G$1" pin="PWM/DP24"/>
+<pinref part="JP3" gate="1" pin="1"/>
+<wire x1="88.9" y1="83.82" x2="81.28" y2="88.9" width="0.1524" layer="91"/>
+<wire x1="81.28" y1="88.9" x2="81.28" y2="109.22" width="0.1524" layer="91"/>
+</segment>
+</net>
+<net name="N$8" class="0">
+<segment>
+<pinref part="JP1" gate="G$1" pin="4"/>
+<pinref part="J3" gate="1" pin="1"/>
+<wire x1="50.8" y1="68.58" x2="53.34" y2="68.58" width="0.1524" layer="91"/>
+<wire x1="53.34" y1="68.58" x2="53.34" y2="73.66" width="0.1524" layer="91"/>
+</segment>
+</net>
